Commit message: Add D405 EOAT refinement and real robot backend

File: src/eoat_description/urdf/rr_00a_b_eoat_no_camera_d405.urdf.xacro (robot description, xacro)
@@ -19,7 +19,7 @@
       mass
       use_nominal_extrinsics:=true
-      d405_x:=0.00905
-      d405_y:=0.04375
-      d405_z:=-0.09105
+      d405_x:=0.00005
+      d405_y:=0.02275
+      d405_z:=-0.10190
       d405_roll:=0
       d405_pitch:=-1.57079632679
@@ -31,4 +31,9 @@
       rpy="${rpy}"
       mass="${mass}"/>
+    <!--
+      Intel's D405 macro origin is the bottom screw frame, not camera_link.
+      These defaults place paint_d405_link at TCP xyz=(0.00905,-0.07640,0.04375),
+      matching the Isaac Sim D405 pose and keeping the rear face on the EOAT bracket.
+    -->
     <xacro:sensor_d405
       parent="${prefix}eoat_no_camera_link"

File: src/eoat_description/urdf/rr_00a_b_eoat_no_camera_d405_standalone.urdf (robot description, URDF)
Before this commit: robot rr_00a_b_eoat_no_camera_d405_standalone, 12 links, 11 joints
Joints:
- joint d405_joint: origin xyz=0.00905 0.04375 -0.09105 rpy=0 -1.57079632679 -1.57079632679 -> xyz=5e-05 0.02275 -0.1019 rpy=0 -1.57079632679 -1.57079632679
